File: PowerSensor/PowerSensor/PowerSensor.kicad_sch (KiCad schematic)
At the start: 11 parts, among them J1 Screw_Terminal_01x02, J2 Screw_Terminal_01x05, J3 Screw_Terminal_01x02, J4 Screw_Terminal_01x02, U1 ACS712ELCTR-20A-T_NRND

Commit message: Change the main project with another project saved on desktop
Parts:
- C1: value C -> 100nF; footprint (none) -> Capacitor_SMD:C_0805_2012Metric
- C2: footprint (none) -> Capacitor_SMD:C_0805_2012Metric
- D1: footprint (none) -> LED_SMD:LED_0805_2012Metric
- J1: footprint TerminalBlock:TerminalBlock_Altech_AK300-2_P5.00mm -> TerminalBlock:TerminalBlock_bornier-2_P5.08mm
- J2: footprint (none) -> TerminalBlock:TerminalBlock_bornier-5_P5.08mm
- J3, J4: footprint (none) -> TerminalBlock:TerminalBlock_bornier-2_P5.08mm
- R1, R2, R3: footprint (none) -> Resistor_SMD:R_0805_2012Metric
Changed lines of the file:
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@@
       (effects (font (size 1.27 1.27)))
     )
-    (property "Footprint" "" (at 246.38 154.178 90)
+    (property "Footprint" "Resistor_SMD:R_0805_2012Metric" (at 246.38 154.178 90)
       (effects (font (size 1.27 1.27)) hide)
     )
@@
       (effects (font (size 1.27 1.27)))
     )
-    (property "Footprint" "" (at 257.81 152.4 0)
+    (property "Footprint" "LED_SMD:LED_0805_2012Metric" (at 257.81 152.4 0)
       (effects (font (size 1.27 1.27)) hide)
     )
@@
       (effects (font (size 1.27 1.27)))
     )
-    (property "Footprint" "" (at 44.45 128.27 0)
+    (property "Footprint" "TerminalBlock:TerminalBlock_bornier-2_P5.08mm" (at 44.45 128.27 0)
       (effects (font (size 1.27 1.27)) hide)
     )
@@
       (effects (font (size 1.27 1.27)) (justify left))
     )
-    (property "Footprint" "" (at 78.232 62.23 90)
+    (property "Footprint" "Resistor_SMD:R_0805_2012Metric" (at 78.232 62.23 90)
       (effects (font (size 1.27 1.27)) hide)
     )
@@
       (effects (font (size 1.27 1.27)))
     )
-    (property "Footprint" "" (at 158.75 127 0)
+    (property "Footprint" "TerminalBlock:TerminalBlock_bornier-5_P5.08mm" (at 158.75 127 0)
       (effects (font (size 1.27 1.27)) hide)
     )
@@
       (effects (font (size 1.27 1.27)) (justify left))
     )
-    (property "Footprint" "" (at 234.6452 71.12 0)
+    (property "Footprint" "Capacitor_SMD:C_0805_2012Metric" (at 234.6452 71.12 0)
       (effects (font (size 1.27 1.27)) hide)
     )
@@
       (effects (font (size 1.27 1.27)) (justify left))
     )
-    (property "Value" "C" (at 232.41 118.11 0)
-      (effects (font (size 1.27 1.27)) (justify left))
-    )
-    (property "Footprint" "" (at 229.5652 120.65 0)
+    (property "Value" "100nF" (at 232.41 118.11 0)
+      (effects (font (size 1.27 1.27)) (justify left))
+    )
+    (property "Footprint" "Capacitor_SMD:C_0805_2012Metric" (at 229.5652 120.65 0)
       (effects (font (size 1.27 1.27)) hide)
     )
@@
       (effects (font (size 1.27 1.27)))
     )
-    (property "Footprint" "" (at 44.45 149.86 0)
+    (property "Footprint" "TerminalBlock:TerminalBlock_bornier-2_P5.08mm" (at 44.45 149.86 0)
       (effects (font (size 1.27 1.27)) hide)
     )
@@
       (effects (font (size 1.27 1.27)))
     )
-    (property "Footprint" "TerminalBlock:TerminalBlock_Altech_AK300-2_P5.00mm" (at 158.75 109.22 0)
+    (property "Footprint" "TerminalBlock:TerminalBlock_bornier-2_P5.08mm" (at 158.75 109.22 0)
       (effects (font (size 1.27 1.27)) hide)
     )
@@
       (effects (font (size 1.27 1.27)) (justify left))
     )
-    (property "Footprint" "" (at 78.232 52.07 90)
-      (effects (font (size 1.27 1.27)) hide)
-    )
+    (property "Footprint" "Resistor_SMD:R_0805_2012Metric" (at 78.232 52.07 90)
+      (effects (font (size 1.27 1.27)) hide)
+    )

Commit message: Add Decoupling Cap 1uF to 5V
Parts:
- added C3: 1uF, Capacitor_SMD:C_0805_2012Metric, symbol Device:C
Connections:
- net +5V: now also C3.1
- net GND: now also C3.2
Changed lines of the file:
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@@
     (stroke (width 0) (type dash_dot))
+  )
+  (wire (pts (xy 248.92 120.65) (xy 248.92 123.19))
+    (stroke (width 0) (type default))
   )
   (wire (pts (xy 53.34 125.73) (xy 59.69 125.73))
@@
   )
   (wire (pts (xy 229.87 59.69) (xy 233.68 59.69))
+    (stroke (width 0) (type default))
+  )
+  (wire (pts (xy 248.92 110.49) (xy 248.92 113.03))
     (stroke (width 0) (type default))
   )
@@
         (path "/273ab69c-9da7-4ae5-8226-b4245c0688ed"
           (reference "#PWR01") (unit 1)
+        )
+      )
+    )
+  )
+  (symbol (lib_id "power:GND") (at 248.92 123.19 0) (unit 1)
+    (in_bom yes) (on_board yes) (dnp no) (fields_autoplaced)
+    (property "Reference" "#PWR011" (at 248.92 129.54 0)
+      (effects (font (size 1.27 1.27)) hide)
+    )
+    (property "Value" "GND" (at 248.92 128.27 0)
+      (effects (font (size 1.27 1.27)))
+    )
+    (property "Footprint" "" (at 248.92 123.19 0)
+      (effects (font (size 1.27 1.27)) hide)
+    )
+    (property "Datasheet" "" (at 248.92 123.19 0)
+      (effects (font (size 1.27 1.27)) hide)
+    )
+    (pin "1")
+    (instances
+      (project "PowerSensor"
+        (path "/273ab69c-9da7-4ae5-8226-b4245c0688ed"
+          (reference "#PWR011") (unit 1)
         )
       )
@@
     )
   )
+  (symbol (lib_id "power:+5V") (at 248.92 110.49 90) (unit 1)
+    (in_bom yes) (on_board yes) (dnp no) (fields_autoplaced)
+    (property "Reference" "#PWR010" (at 252.73 110.49 0)
+      (effects (font (size 1.27 1.27)) hide)
+    )
+    (property "Value" "+5V" (at 245.11 110.49 90)
+      (effects (font (size 1.27 1.27)) (justify left))
+    )
+    (property "Footprint" "" (at 248.92 110.49 0)
+      (effects (font (size 1.27 1.27)) hide)
+    )
+    (property "Datasheet" "" (at 248.92 110.49 0)
+      (effects (font (size 1.27 1.27)) hide)
+    )
+    (pin "1")
+    (instances
+      (project "PowerSensor"
+        (path "/273ab69c-9da7-4ae5-8226-b4245c0688ed"
+          (reference "#PWR010") (unit 1)
+        )
+      )
+    )
+  )
   (symbol (lib_id "Device:R") (at 80.01 52.07 0) (unit 1)
     (in_bom yes) (on_board yes) (dnp no) (fields_autoplaced)
@@
         )
       )
+    )
+  )
+  (symbol (lib_id "Device:C") (at 248.92 116.84 0) (unit 1)
+    (in_bom yes) (on_board yes) (dnp no) (fields_autoplaced)
+    (property "Reference" "C3" (at 252.73 115.57 0)
+      (effects (font (size 1.27 1.27)) (justify left))
+    )
+    (property "Value" "1uF" (at 252.73 118.11 0)
+      (effects (font (size 1.27 1.27)) (justify left))
+    )
+    (property "Footprint" "Capacitor_SMD:C_0805_2012Metric" (at 249.8852 120.65 0)
+      (effects (font (size 1.27 1.27)) hide)
+    )
+    (property "Datasheet" "~" (at 248.92 116.84 0)
+      (effects (font (size 1.27 1.27)) hide)
+    )
+    (pin "1")
+    (pin "2")
+    (instances
+      (project "PowerSensor"
+        (path "/273ab69c-9da7-4ae5-8226-b4245c0688ed"
+          (reference "C3") (unit 1)
+        )
+      )

Commit message: Add decupling Cap to 5V
Parts:
- added C4: 1uF, Capacitor_SMD:C_0805_2012Metric, symbol Device:C
Connections:
- net +5V: now also C4.1
- net GND: now also C4.2
Changed lines of the file:
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@@
+    (stroke (width 0) (type default))
+  )
+  (wire (pts (xy 266.7 119.38) (xy 266.7 121.92))
     (stroke (width 0) (type default))
   )
@@
   )
   (wire (pts (xy 80.01 44.45) (xy 80.01 48.26))
+    (stroke (width 0) (type default))
+  )
+  (wire (pts (xy 266.7 109.22) (xy 266.7 111.76))
     (stroke (width 0) (type default))
   )
@@
         (path "/273ab69c-9da7-4ae5-8226-b4245c0688ed"
           (reference "J3") (unit 1)
+        )
+      )
+    )
+  )
+  (symbol (lib_id "power:+5V") (at 266.7 109.22 90) (unit 1)
+    (in_bom yes) (on_board yes) (dnp no) (fields_autoplaced)
+    (property "Reference" "#PWR012" (at 270.51 109.22 0)
+      (effects (font (size 1.27 1.27)) hide)
+    )
+    (property "Value" "+5V" (at 262.89 109.22 90)
+      (effects (font (size 1.27 1.27)) (justify left))
+    )
+    (property "Footprint" "" (at 266.7 109.22 0)
+      (effects (font (size 1.27 1.27)) hide)
+    )
+    (property "Datasheet" "" (at 266.7 109.22 0)
+      (effects (font (size 1.27 1.27)) hide)
+    )
+    (pin "1")
+    (instances
+      (project "PowerSensor"
+        (path "/273ab69c-9da7-4ae5-8226-b4245c0688ed"
+          (reference "#PWR012") (unit 1)
+        )
+      )
+    )
+  )
+  (symbol (lib_id "power:GND") (at 266.7 121.92 0) (unit 1)
+    (in_bom yes) (on_board yes) (dnp no) (fields_autoplaced)
+    (property "Reference" "#PWR013" (at 266.7 128.27 0)
+      (effects (font (size 1.27 1.27)) hide)
+    )
+    (property "Value" "GND" (at 266.7 127 0)
+      (effects (font (size 1.27 1.27)))
+    )
+    (property "Footprint" "" (at 266.7 121.92 0)
+      (effects (font (size 1.27 1.27)) hide)
+    )
+    (property "Datasheet" "" (at 266.7 121.92 0)
+      (effects (font (size 1.27 1.27)) hide)
+    )
+    (pin "1")
+    (instances
+      (project "PowerSensor"
+        (path "/273ab69c-9da7-4ae5-8226-b4245c0688ed"
+          (reference "#PWR013") (unit 1)
         )
       )
@@
         )
       )
+    )
+  )
+  (symbol (lib_id "Device:C") (at 266.7 115.57 0) (unit 1)
+    (in_bom yes) (on_board yes) (dnp no) (fields_autoplaced)
+    (property "Reference" "C4" (at 270.51 114.3 0)
+      (effects (font (size 1.27 1.27)) (justify left))
+    )
+    (property "Value" "1uF" (at 270.51 116.84 0)
+      (effects (font (size 1.27 1.27)) (justify left))
+    )
+    (property "Footprint" "Capacitor_SMD:C_0805_2012Metric" (at 267.6652 119.38 0)
+      (effects (font (size 1.27 1.27)) hide)
+    )
+    (property "Datasheet" "~" (at 266.7 115.57 0)
+      (effects (font (size 1.27 1.27)) hide)
+    )
+    (pin "1")
+    (pin "2")
+    (instances
+      (project "PowerSensor"
+        (path "/273ab69c-9da7-4ae5-8226-b4245c0688ed"
+          (reference "C4") (unit 1)
+        )
+      )
