File: PowerSensor/PowerSensor/PowerSensor.kicad_pcb (KiCad board)
At the start: 2 copper layers, 35.6 x 22.6 mm, 12 parts, among them J1 Current Sens, J3 BAT+, J4 BAT-, J5 Screw_Terminal_01x04, U1 ACS712ELCTR-20A-T_NRND

Commit message: optimization
Routing:
- net GND: track 25.8 -> 28.7 mm
- net IN+: track 14.8 -> 13.6 mm
- net IN-: track 8.64 -> 9.45 mm
- net Battery(+): track 14.7 -> 15.3 mm
- net Battery(-): track 12.1 -> 12.7 mm
Other:
- board text added: "BAT+"
- board text added: "BAT-"
Changed lines of the file:
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@@
   )
   (setup
+    (stackup
+      (layer "F.SilkS" (type "Top Silk Screen"))
+      (layer "F.Paste" (type "Top Solder Paste"))
+      (layer "F.Mask" (type "Top Solder Mask") (thickness 0.01))
+      (layer "F.Cu" (type "copper") (thickness 0.035))
+      (layer "dielectric 1" (type "core") (thickness 1.51) (material "FR4") (epsilon_r 4.5) (loss_tangent 0.02))
+      (layer "B.Cu" (type "copper") (thickness 0.035))
+      (layer "B.Mask" (type "Bottom Solder Mask") (thickness 0.01))
+      (layer "B.Paste" (type "Bottom Solder Paste"))
+      (layer "B.SilkS" (type "Bottom Silk Screen"))
+      (copper_finish "None")
+      (dielectric_constraints no)
+    )
     (pad_to_mask_clearance 0)
     (pcbplotparams
@@
     (property "ki_keywords" "screw terminal")
     (attr through_hole)
-    (fp_text reference "J3" (at 2.54 -5.08 90) (layer "F.SilkS")
+    (fp_text reference "J3" (at -0.52 -2.6 90) (layer "F.SilkS")
         (effects (font (size 1 1) (thickness 0.15)))
     )
@@
     (property "ki_keywords" "LED diode")
     (attr smd)
-    (fp_text reference "D1" (at 2.7375 0 90) (layer "F.SilkS")
+    (fp_text reference "D1" (at -2.7375 -0.2 90) (layer "F.SilkS")
         (effects (font (size 1 1) (thickness 0.15)))
     )
@@
     (property "ki_keywords" "620-1190-1-ND")
     (attr smd)
-    (fp_text reference "U1" (at 0 -3.4) (layer "F.SilkS")
+    (fp_text reference "U1" (at -4.8 -1.6) (layer "F.SilkS")
         (effects (font (size 1 1) (thickness 0.15)))
     )
@@
     (property "ki_keywords" "screw terminal")
     (attr through_hole)
-    (fp_text reference "J5" (at 7.6 -4.8 90) (layer "F.SilkS")
+    (fp_text reference "J5" (at 7.64 -2.6 90) (layer "F.SilkS")
         (effects (font (size 1 1) (thickness 0.15)))
     )
@@
     (property "ki_keywords" "screw terminal")
     (attr through_hole)
-    (fp_text reference "J4" (at 2.54 -5.08 90) (layer "F.SilkS")
+    (fp_text reference "J4" (at 0.48 -2.8 90) (layer "F.SilkS")
         (effects (font (size 1 1) (thickness 0.15)))
     )
@@
   (gr_rect (start 91.4 81.2) (end 127 103.8)
     (stroke (width 0.1) (type default)) (fill none) (layer "Edge.Cuts"))
-  (gr_text "ISens" (at 123 94.8) (layer "F.SilkS")
-    (effects (font (size 0.75 0.75) (thickness 0.15)) (justify left bottom))
-  )
-  (gr_text "GND" (at 123.2 84.8) (layer "F.SilkS")
+  (gr_text "ISens" (at 125.2 97 90) (layer "F.SilkS")
     (effects (font (size 1 1) (thickness 0.15)) (justify left bottom))
   )
-  (gr_text "+5V" (at 123 90) (layer "F.SilkS")
+  (gr_text "GND" (at 125.2 85.8 90) (layer "F.SilkS")
     (effects (font (size 1 1) (thickness 0.15)) (justify left bottom))
   )
-  (gr_text "VSens" (at 123 99.8) (layer "F.SilkS")
-    (effects (font (size 0.75 0.75) (thickness 0.15)) (justify left bottom))
+  (gr_text "+5V" (at 125.2 91.2 90) (layer "F.SilkS")
+    (effects (font (size 1 1) (thickness 0.15)) (justify left bottom))
+  )
+  (gr_text "BAT+" (at 100 82.8) (layer "F.SilkS")
+    (effects (font (size 1 1) (thickness 0.25) bold) (justify left bottom))
+  )
+  (gr_text "BAT-" (at 100.2 93.6) (layer "F.SilkS")
+    (effects (font (size 1 1) (thickness 0.25) bold) (justify left bottom))
+  )
+  (gr_text "VSens" (at 125.2 103 90) (layer "F.SilkS")
+    (effects (font (size 1 1) (thickness 0.15)) (justify left bottom))
   )
   (segment (start 111.675 94.105) (end 113.295 94.105) (width 0.25) (layer "F.Cu") (net 1))
+  (segment (start 118.8 84.36) (end 118.04 83.6) (width 1) (layer "F.Cu") (net 1))
+  (segment (start 105.2 85.8) (end 105.2 83.6) (width 0.25) (layer "F.Cu") (net 1))
   (segment (start 113.295 94.105) (end 113.6 93.8) (width 0.25) (layer "F.Cu") (net 1))
-  (segment (start 109.8 84.36) (end 105.2 84.36) (width 0.25) (layer "F.Cu") (net 1))
-  (segment (start 112.2 84.36) (end 109.8 84.36) (width 0.25) (layer "F.Cu") (net 1))
   (segment (start 102.84 84.36) (end 102.8 84.4) (width 0.25) (layer "F.Cu") (net 1))
-  (segment (start 112.2 85.8) (end 112.2 84.36) (width 0.25) (layer "F.Cu") (net 1))
-  (segment (start 109.8 85.8) (end 109.8 84.36) (width 0.25) (layer "F.Cu") (net 1))
-  (segment (start 105.2 85.8) (end 105.2 84.36) (width 0.25) (layer "F.Cu") (net 1))
-  (segment (start 118.8 84.36) (end 112.2 84.36) (width 0.25) (layer "F.Cu") (net 1))
+  (segment (start 112.2 85.8) (end 112.2 83.6) (width 0.25) (layer "F.Cu") (net 1))
   (segment (start 102.8 84.4) (end 102.8 85.8) (width 0.25) (layer "F.Cu") (net 1))
   (segment (start 113.6 92.8) (end 113.6 94.8) (width 0.25) (layer "F.Cu") (net 1))
-  (segment (start 105.2 84.36) (end 102.84 84.36) (width 0.25) (layer "F.Cu") (net 1))
+  (segment (start 109.8 85.8) (end 109.8 83.6) (width 0.25) (layer "F.Cu") (net 1))
+  (segment (start 118.04 83.6) (end 103.6 83.6) (width 1) (layer "F.Cu") (net 1))
+  (segment (start 103.6 83.6) (end 102.84 84.36) (width 1) (layer "F.Cu") (net 1))
   (via (at 113.6 93.8) (size 0.8) (drill 0.4) (layers "F.Cu" "B.Cu") (free) (net 1))
   (via (at 113.6 94.8) (size 0.8) (drill 0.4) (layers "F.Cu" "B.Cu") (free) (net 1))
@@
   (segment (start 105.2 87.4) (end 105.2 87.675) (width 0.25) (layer "F.Cu") (net 2))
   (segment (start 106.8 85.8) (end 105.2 87.4) (width 0.25) (layer "F.Cu") (net 2))
-  (segment (start 111.74 99.12) (end 106.725 94.105) (width 0.2) (layer "F.Cu") (net 3))
+  (segment (start 111.74 99.12) (end 111.74 97.74) (width 1) (layer "F.Cu") (net 3))
+  (segment (start 108.105 94.105) (end 106.725 94.105) (width 1) (layer "F.Cu") (net 3))
+  (segment (start 111.74 97.74) (end 108.105 94.105) (width 1) (layer "F.Cu") (net 3))
   (segment (start 111.74 99.4) (end 111.74 99.12) (width 0.2) (layer "F.Cu") (net 3))
-  (segment (start 106.725 94.105) (end 106.725 92.835) (width 0.2) (layer "F.Cu") (net 3))
-  (segment (start 103.905 90.295) (end 106.725 90.295) (width 0.2) (layer "F.Cu") (net 4))
-  (segment (start 106.725 90.295) (end 106.725 91.565) (width 0.2) (layer "F.Cu") (net 4))
-  (segment (start 103.4 90.8) (end 103.905 90.295) (width 0.2) (layer "F.Cu") (net 4))
-  (segment (start 106.66 99.4) (end 103.4 96.14) (width 0.2) (layer "F.Cu") (net 4))
-  (segment (start 103.4 96.14) (end 103.4 90.8) (width 0.2) (layer "F.Cu") (net 4))
-  (segment (start 97.8325 102.1125) (end 95.8 100.08) (width 0.25) (layer "F.Cu") (net 5))
-  (segment (start 95.8 95) (end 95.8 100.08) (width 0.25) (layer "F.Cu") (net 5))
-  (segment (start 102 102.1125) (end 97.8325 102.1125) (width 0.25) (layer "F.Cu") (net 5))
+  (segment (start 106.725 94.105) (end 106.725 92.835) (width 1) (layer "F.Cu") (net 3))
+  (segment (start 106.66 99.4) (end 104.2 96.94) (width 1) (layer "F.Cu") (net 4))
+  (segment (start 104.705 90.295) (end 106.725 90.295) (width 1) (layer "F.Cu") (net 4))
+  (segment (start 104.2 90.8) (end 104.705 90.295) (width 1) (layer "F.Cu") (net 4))
+  (segment (start 104.2 96.94) (end 104.2 90.8) (width 1) (layer "F.Cu") (net 4))
+  (segment (start 106.725 90.295) (end 106.725 91.565) (width 1) (layer "F.Cu") (net 4))
+  (segment (start 102.4 102.6) (end 98.32 102.6) (width 2) (layer "F.Cu") (net 5))
+  (segment (start 95.8 95) (end 95.8 100.08) (width 2) (layer "F.Cu") (net 5))
+  (segment (start 98.32 102.6) (end 95.8 100.08) (width 2) (layer "F.Cu") (net 5))
   (segment (start 109.8 90) (end 110.095 90.295) (width 0.25) (layer "F.Cu") (net 6))
   (segment (start 115.04 89.44) (end 113.3 87.7) (width 0.25) (layer "F.Cu") (net 6))
@@
   (segment (start 115.845 91.565) (end 118.8 94.52) (width 0.25) (layer "F.Cu") (net 7))
   (segment (start 111.675 91.565) (end 115.845 91.565) (width 0.25) (layer "F.Cu") (net 7))
-  (segment (start 118.8 99.6) (end 116.6 99.6) (width 0.25) (layer "F.Cu") (net 8))
-  (segment (start 114.2 102) (end 104.8 102) (width 0.25) (layer "F.Cu") (net 8))
-  (segment (start 102 99.2) (end 102 100.2875) (width 0.25) (layer "F.Cu") (net 8))
-  (segment (start 102 98.3125) (end 102 99.2) (width 0.25) (layer "F.Cu") (net 8))
-  (segment (start 116.6 99.6) (end 114.2 102) (width 0.25) (layer "F.Cu") (net 8))
-  (segment (start 104.8 102) (end 102 99.2) (width 0.25) (layer "F.Cu") (net 8))
-  (segment (start 95.8 84.4) (end 95.8 89.48) (width 0.25) (layer "F.Cu") (net 9))
-  (segment (start 102 96.4875) (end 102 95.68) (width 0.25) (layer "F.Cu") (net 9))
-  (segment (start 102 95.68) (end 95.8 89.48) (width 0.25) (layer "F.Cu") (net 9))
+  (segment (start 113.8 102.4) (end 116.6 99.6) (width 1) (layer "F.Cu") (net 8))
+  (segment (start 116.6 99.6) (end 118.8 99.6) (width 1) (layer "F.Cu") (net 8))
+  (segment (start 102 99.3) (end 103.3 99.3) (width 1) (layer "F.Cu") (net 8))
+  (segment (start 106.4 102.4) (end 113.8 102.4) (width 1) (layer "F.Cu") (net 8))
+  (segment (start 102 98.3125) (end 102 100.2875) (width 1) (layer "F.Cu") (net 8))
+  (segment (start 103.3 99.3) (end 106.4 102.4) (width 1) (layer "F.Cu") (net 8))
+  (segment (start 95.8 84.4) (end 95.8 89.48) (width 2) (layer "F.Cu") (net 9))
+  (segment (start 100 91.6) (end 97.88 89.48) (width 2) (layer "F.Cu") (net 9))
+  (segment (start 97.88 89.48) (end 95.8 89.48) (width 2) (layer "F.Cu") (net 9))
+  (segment (start 100 94.2) (end 100 91.6) (width 2) (layer "F.Cu") (net 9))
+  (segment (start 101.8 96) (end 100 94.2) (width 2) (layer "F.Cu") (net 9))
   (segment (start 109.35 89.95) (end 109.35 92.75) (width 0.25) (layer "F.Cu") (net 10))
   (segment (start 102.8 87.7) (end 102.8 89) (width 0.25) (layer "F.Cu") (net 10))

Commit message: PCB optimization 2
Parts:
- moved R1 1.49 mm to (102.0, 95.9)
Routing:
- net Vsens: track 21.2 -> 25.7 mm
- net VIOUT: track 8.35 -> 9.42 mm
Changed lines of the file:
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@@
   )
   (footprint "Resistor_SMD:R_0805_2012Metric" (layer "F.Cu")
-    (at 102 97.4 -90)
+    (at 102 95.9125 -90)
     (descr "Resistor SMD 0805 (2012 Metric), square (rectangular) end terminal, IPC_7351 nominal, (Body size source: IPC-SM-782 page 72, https://www.pcb-3d.com/wordpress/wp-content/uploads/ipc-sm-782a_amendment_1_and_2.pdf), generated with kicad-footprint-generator")
     (tags "resistor")
@@
     (effects (font (size 1 1) (thickness 0.15)) (justify left bottom))
   )
+  (segment (start 102.9 83.575) (end 102.84 83.635) (width 1) (layer "F.Cu") (net 1))
   (segment (start 111.675 94.105) (end 113.295 94.105) (width 0.25) (layer "F.Cu") (net 1))
+  (segment (start 105.2 85.8) (end 105.2 83.6) (width 1) (layer "F.Cu") (net 1))
+  (segment (start 113.295 94.105) (end 113.6 93.8) (width 0.25) (layer "F.Cu") (net 1))
   (segment (start 118.8 84.36) (end 118.04 83.6) (width 1) (layer "F.Cu") (net 1))
-  (segment (start 105.2 85.8) (end 105.2 83.6) (width 0.25) (layer "F.Cu") (net 1))
-  (segment (start 113.295 94.105) (end 113.6 93.8) (width 0.25) (layer "F.Cu") (net 1))
   (segment (start 102.84 84.36) (end 102.8 84.4) (width 0.25) (layer "F.Cu") (net 1))
-  (segment (start 112.2 85.8) (end 112.2 83.6) (width 0.25) (layer "F.Cu") (net 1))
-  (segment (start 102.8 84.4) (end 102.8 85.8) (width 0.25) (layer "F.Cu") (net 1))
+  (segment (start 112.2 85.8) (end 112.2 83.6) (width 1) (layer "F.Cu") (net 1))
+  (segment (start 102.925 83.6) (end 102.9 83.575) (width 1) (layer "F.Cu") (net 1))
+  (segment (start 102.8 84.4) (end 102.8 85.8) (width 1) (layer "F.Cu") (net 1))
   (segment (start 113.6 92.8) (end 113.6 94.8) (width 0.25) (layer "F.Cu") (net 1))
-  (segment (start 109.8 85.8) (end 109.8 83.6) (width 0.25) (layer "F.Cu") (net 1))
-  (segment (start 118.04 83.6) (end 103.6 83.6) (width 1) (layer "F.Cu") (net 1))
-  (segment (start 103.6 83.6) (end 102.84 84.36) (width 1) (layer "F.Cu") (net 1))
+  (segment (start 118.04 83.6) (end 102.925 83.6) (width 1) (layer "F.Cu") (net 1))
+  (segment (start 109.8 85.8) (end 109.8 83.6) (width 1) (layer "F.Cu") (net 1))
+  (segment (start 102.84 83.635) (end 102.84 84.36) (width 1) (layer "F.Cu") (net 1))
   (via (at 113.6 93.8) (size 0.8) (drill 0.4) (layers "F.Cu" "B.Cu") (free) (net 1))
   (via (at 113.6 94.8) (size 0.8) (drill 0.4) (layers "F.Cu" "B.Cu") (free) (net 1))
@@
   (segment (start 112.2 87.7) (end 109.8 87.7) (width 0.25) (layer "F.Cu") (net 6))
   (segment (start 109.8 87.7) (end 109.8 90) (width 0.25) (layer "F.Cu") (net 6))
-  (segment (start 115.845 91.565) (end 118.8 94.52) (width 0.25) (layer "F.Cu") (net 7))
-  (segment (start 111.675 91.565) (end 115.845 91.565) (width 0.25) (layer "F.Cu") (net 7))
-  (segment (start 113.8 102.4) (end 116.6 99.6) (width 1) (layer "F.Cu") (net 8))
-  (segment (start 116.6 99.6) (end 118.8 99.6) (width 1) (layer "F.Cu") (net 8))
-  (segment (start 102 99.3) (end 103.3 99.3) (width 1) (layer "F.Cu") (net 8))
-  (segment (start 106.4 102.4) (end 113.8 102.4) (width 1) (layer "F.Cu") (net 8))
-  (segment (start 102 98.3125) (end 102 100.2875) (width 1) (layer "F.Cu") (net 8))
-  (segment (start 103.3 99.3) (end 106.4 102.4) (width 1) (layer "F.Cu") (net 8))
+  (segment (start 115.4 91.565) (end 115.4 93.4) (width 0.6) (layer "F.Cu") (net 7))
+  (segment (start 116.52 94.52) (end 118.8 94.52) (width 0.6) (layer "F.Cu") (net 7))
+  (segment (start 111.675 91.565) (end 115.4 91.565) (width 0.6) (layer "F.Cu") (net 7))
+  (segment (start 115.4 93.4) (end 116.52 94.52) (width 0.6) (layer "F.Cu") (net 7))
+  (segment (start 115.35 99.6) (end 118.8 99.6) (width 1) (layer "F.Cu") (net 8))
+  (segment (start 105.7 102.4) (end 115.35 102.4) (width 1) (layer "F.Cu") (net 8))
+  (segment (start 115.35 102.4) (end 115.35 99.6) (width 1) (layer "F.Cu") (net 8))
+  (segment (start 103.6 98.5) (end 103.7 98.6) (width 1) (layer "F.Cu") (net 8))
+  (segment (start 103.7 98.6) (end 103.7 100.4) (width 1) (layer "F.Cu") (net 8))
+  (segment (start 102 96.825) (end 102 100.2875) (width 1) (layer "F.Cu") (net 8))
+  (segment (start 102 98.5) (end 103.6 98.5) (width 1) (layer "F.Cu") (net 8))
+  (segment (start 103.7 100.4) (end 105.7 102.4) (width 1) (layer "F.Cu") (net 8))
   (segment (start 95.8 84.4) (end 95.8 89.48) (width 2) (layer "F.Cu") (net 9))
-  (segment (start 100 91.6) (end 97.88 89.48) (width 2) (layer "F.Cu") (net 9))
-  (segment (start 97.88 89.48) (end 95.8 89.48) (width 2) (layer "F.Cu") (net 9))
-  (segment (start 100 94.2) (end 100 91.6) (width 2) (layer "F.Cu") (net 9))
-  (segment (start 101.8 96) (end 100 94.2) (width 2) (layer "F.Cu") (net 9))
-  (segment (start 109.35 89.95) (end 109.35 92.75) (width 0.25) (layer "F.Cu") (net 10))
+  (segment (start 99.68 89.48) (end 95.8 89.48) (width 2) (layer "F.Cu") (net 9))
+  (segment (start 102 94.5) (end 102 91.8) (width 2) (layer "F.Cu") (net 9))
+  (segment (start 102 91.8) (end 99.68 89.48) (width 2) (layer "F.Cu") (net 9))
+  (segment (start 108.5 89) (end 108.9 89.4) (width 0.25) (layer "F.Cu") (net 10))
+  (segment (start 102.8 89) (end 108.5 89) (width 0.25) (layer "F.Cu") (net 10))
+  (segment (start 109.435 92.835) (end 111.675 92.835) (width 0.25) (layer "F.Cu") (net 10))
+  (segment (start 108.9 89.4) (end 108.9 92.3) (width 0.25) (layer "F.Cu") (net 10))
   (segment (start 102.8 87.7) (end 102.8 89) (width 0.25) (layer "F.Cu") (net 10))
-  (segment (start 108.4 89) (end 109.35 89.95) (width 0.25) (layer "F.Cu") (net 10))
-  (segment (start 102.8 89) (end 108.4 89) (width 0.25) (layer "F.Cu") (net 10))
-  (segment (start 109.435 92.835) (end 111.675 92.835) (width 0.25) (layer "F.Cu") (net 10))
-  (segment (start 109.35 92.75) (end 109.435 92.835) (width 0.25) (layer "F.Cu") (net 10))
+  (segment (start 108.9 92.3) (end 109.435 92.835) (width 0.25) (layer "F.Cu") (net 10))
   (zone (net 1) (net_name "GND") (layer "B.Cu") (hatch edge 0.5)
-    (connect_pads (clearance 0.5))
+    (connect_pads yes (clearance 0.5))
     (min_thickness 0.25) (filled_areas_thickness no)
     (fill yes (thermal_gap 0.5) (thermal_bridge_width 0.5))
